File: HW_STM32/CMSIS-DAP-X893/CMSIS-DAP.V1.brd (EAGLE design)
At the start: 31.4 x 13.6 mm, 36 parts, among them IC1 STM32F103CBT6, J2 USB-4-AP-1P, J3 USB-4-A-SMD, Q1 8M, U7 TPS73033, X1 USB-SMD

Commit message: Fix RESET pin
Other:
- board text added: "Version 1"
Changed lines of the file:
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@@
 <text x="-2.9" y="3.6" size="1.27" layer="51" ratio="15" rot="R90">MiniUSB</text>
 <text x="-4.9" y="2.6" size="1.27" layer="51" ratio="15" rot="R90">USB-A or</text>
+<text x="0.2" y="22.2" size="2" layer="49" ratio="15">Version 1</text>
 </plain>
 <attributes>
